Commit message: fixed _ issue in prefix

File: urdf/robot_kitchen.macro.xacro (robot description, xacro)
@@ -37,5 +37,5 @@
         </link>
         <!-- Reference -->
-        <link name="${prefix}_kitchen_reference"/>
+        <link name="${prefix}kitchen_reference"/>
         <!-- Parent to Kitchen -->
         <joint name="${parent}to_kitchen" type="fixed">
@@ -48,5 +48,5 @@
         <joint name="${prefix}kitchen_to_kitchen_reference" type="fixed">
             <parent link="${prefix}kitchen"/>
-            <child link="${prefix}_kitchen_reference"/>
+            <child link="${prefix}kitchen_reference"/>
             <origin xyz ="0 ${-0.13-0.207/2.} 0" rpy="0 0 0"/>
         </joint>

Commit message: changed aurora kitchen params

File: urdf/robot_kitchen.macro.xacro (robot description, xacro)
@@ -7,6 +7,6 @@
         <xacro:property name="kitchen_width_electrolux" value="1.082"/>
         <xacro:property name="kitchen_height_electrolux" value="0.89599"/>
-        <xacro:property name="kitchen_length_aurora" value="2."/>
-        <xacro:property name="kitchen_width_aurora" value="1.2"/>
+        <xacro:property name="kitchen_length_aurora" value="2.775"/>
+        <xacro:property name="kitchen_width_aurora" value="1.137"/>
         <xacro:property name="kitchen_height_aurora" value="1.1"/>
         <xacro:if value="${model == 'electrolux'}">
@@ -15,5 +15,5 @@
             <xacro:property name="kitchen_height" value="${kitchen_height_electrolux}"/>
         </xacro:if>
-        <xacro:unless value="${model == 'aurora'}">
+        <xacro:unless value="${model == 'electrolux'}">
             <xacro:property name="kitchen_length" value="${kitchen_length_aurora}"/>
             <xacro:property name="kitchen_width" value="${kitchen_width_aurora}"/>

Commit message: switched from stl to dae with textures

File: urdf/robot_kitchen.macro.xacro (robot description, xacro)
@@ -24,5 +24,5 @@
             <visual>
                 <geometry>
-                    <mesh filename="package://robot_kitchen_description/meshes/kitchen_${model}.stl"/>
+                    <mesh filename="package://robot_kitchen_description/meshes/kitchen_${model}.dae"/>
                 </geometry>
             </visual>

Commit message: first

File: urdf/robot_kitchen.macro.xacro (robot description, xacro)
@@ -10,4 +10,5 @@
         <xacro:property name="kitchen_width_aurora" value="1.137"/>
         <xacro:property name="kitchen_height_aurora" value="1.1"/>
+        <xacro:property name="kitchen_mass" value="1000"/>
         <xacro:if value="${model == 'electrolux'}">
             <xacro:property name="kitchen_length" value="${kitchen_length_electrolux}"/>
@@ -20,4 +21,22 @@
             <xacro:property name="kitchen_height" value="${kitchen_height_aurora}"/>
         </xacro:unless>
+        <xacro:macro name="cylinder_inertial" params="radius length mass *origin">
+            <inertial>
+            <mass value="${mass}" />
+            <xacro:insert_block name="origin" />
+            <inertia ixx="${0.0833333 * mass * (3 * radius * radius + length * length)}" ixy="0.0" ixz="0.0"
+            iyy="${0.0833333 * mass * (3 * radius * radius + length * length)}" iyz="0.0"
+            izz="${0.5 * mass * radius * radius}" />
+            </inertial>
+        </xacro:macro>
+        <xacro:macro name="box_inertial" params="length width height mass">
+            <inertial>
+            <mass value="${mass}" />
+            <inertia ixx="${0.0833333 * mass * (width * width + height * height)}" ixy="0.0" ixz="0.0"
+            iyy="${0.0833333 * mass * (length * length + height * height)}" iyz="0.0"
+            izz="${0.083 * length * length + width * width}" />
+            </inertial>
+        </xacro:macro>
+        <static>true</static>
         <!-- Kitchen -->
         <link name="${prefix}kitchen">
@@ -27,5 +46,4 @@
                 </geometry>
             </visual>
-            <!--
             <collision>
                 <origin xyz="${kitchen_length/2.} ${-kitchen_width/2.} ${-kitchen_height/2.}" rpy="0 0 0"/>
@@ -34,6 +52,9 @@
                 </geometry>
             </collision>
-            -->
+            <box_inertial length="${kitchen_length}" width="${kitchen_width}" height="${kitchen_height}" mass="${kitchen_mass}" />
         </link>
+        <gazebo reference="${prefix}kitchen">
+            <material>Gazebo/Gray</material>
+        </gazebo>
         <!-- Reference -->
         <link name="${prefix}kitchen_reference"/>
